Commit message: f**k this

File: Control/panda/src/panda_description/urdf/panda_desc.urdf.xacro (robot description, xacro)
@@ -270,5 +270,5 @@
         </collision>
         <inertial>
-          <origin xyz="0 0 0" rpy="0 0 0" />
+          <origin xyz="0 0 0" rpy="5 0 0" />
           <mass value="0.15"/>
           <inertia ixx="2.375E-6" iyy="2.375E-6" izz="7.5E-7" ixy="0" ixz="0" iyz="0"/>

File: Control/panda/src/panda_description/urdf/ros2_control.xacro (robot description, xacro)
@@ -62,4 +62,11 @@
                 <state_interface name="velocity"/>
             </joint>
+            <joint name="panda_finger_joint2">
+                <command_interface name="position"/>
+                <state_interface name="position">
+                  <param name="initial_value">0.0</param>
+                </state_interface>
+                <state_interface name="velocity"/>
+            </joint>
         </ros2_control>
 </robot>
