Commit message: The legend of Po

File: Control/panda/src/panda_description/urdf/panda.urdf.xacro (robot description, xacro)
@@ -8,27 +8,27 @@
         <visual>
             <geometry>
-                <mesh filename="file://$(find moveit_resources_panda_description)/meshes/visual/link0.dae" />
-            </geometry>
-        </visual>
-        <collision>
-            <geometry>
-                <mesh filename="file://$(find moveit_resources_panda_description)/meshes/collision/link0.stl" />
-            </geometry>
-        </collision>
-        <inertial>
-          <origin xyz="-0.041018 -0.00014 0.049974" rpy="0 0 0" />
-          <mass value="0.629769"/>
-          <inertia ixx="0.00315" iyy="0.00388" izz="0.004285" ixy="8.2904E-7" ixz="0.00015" iyz="8.2299E-6"/>
-        </inertial>
+                <mesh filename="file://$(find panda_description)/meshes/visual/link0.dae" />
+            </geometry>
+        </visual>
+        <collision>
+            <geometry>
+                <mesh filename="file://$(find panda_description)/meshes/collision/link0.stl" />
+            </geometry>
+        </collision>
+        <!-- <inertial> -->
+          <!-- <origin xyz="-0.041018 -0.00014 0.049974" rpy="0 0 0" /> -->
+          <!-- <mass value="0.629769"/> -->
+          <!-- <inertia ixx="0.00315" iyy="0.00388" izz="0.004285" ixy="8.2904E-7" ixz="0.00015" iyz="8.2299E-6"/> -->
+        <!-- </inertial> -->
     </link>
     <link name="panda_link1">
         <visual>
             <geometry>
-                <mesh filename="file://$(find moveit_resources_panda_description)/meshes/visual/link1.dae" />
-            </geometry>
-        </visual>
-        <collision>
-            <geometry>
-                <mesh filename="file://$(find moveit_resources_panda_description)/meshes/collision/link1.stl" />
+                <mesh filename="file://$(find panda_description)/meshes/visual/link1.dae" />
+            </geometry>
+        </visual>
+        <collision>
+            <geometry>
+                <mesh filename="file://$(find panda_description)/meshes/collision/link1.stl" />
             </geometry>
         </collision>
@@ -51,10 +51,10 @@
         <visual>
             <geometry>
-                <mesh filename="file://$(find moveit_resources_panda_description)/meshes/visual/link2.dae" />
-            </geometry>
-        </visual>
-        <collision>
-            <geometry>
-                <mesh filename="file://$(find moveit_resources_panda_description)/meshes/collision/link2.stl" />
+                <mesh filename="file://$(find panda_description)/meshes/visual/link2.dae" />
+            </geometry>
+        </visual>
+        <collision>
+            <geometry>
+                <mesh filename="file://$(find panda_description)/meshes/collision/link2.stl" />
             </geometry>
         </collision>
@@ -77,10 +77,10 @@
         <visual>
             <geometry>
-                <mesh filename="file://$(find moveit_resources_panda_description)/meshes/visual/link3.dae" />
-            </geometry>
-        </visual>
-        <collision>
-            <geometry>
-                <mesh filename="file://$(find moveit_resources_panda_description)/meshes/collision/link3.stl" />
+                <mesh filename="file://$(find panda_description)/meshes/visual/link3.dae" />
+            </geometry>
+        </visual>
+        <collision>
+            <geometry>
+                <mesh filename="file://$(find panda_description)/meshes/collision/link3.stl" />
             </geometry>
         </collision>
@@ -103,10 +103,10 @@
         <visual>
             <geometry>
-                <mesh filename="file://$(find moveit_resources_panda_description)/meshes/visual/link4.dae" />
-            </geometry>
-        </visual>
-        <collision>
-            <geometry>
-                <mesh filename="file://$(find moveit_resources_panda_description)/meshes/collision/link4.stl" />
+                <mesh filename="file://$(find panda_description)/meshes/visual/link4.dae" />
+            </geometry>
+        </visual>
+        <collision>
+            <geometry>
+                <mesh filename="file://$(find panda_description)/meshes/collision/link4.stl" />
             </geometry>
         </collision>
@@ -129,10 +129,10 @@
         <visual>
             <geometry>
-                <mesh filename="file://$(find moveit_resources_panda_description)/meshes/visual/link5.dae" />
-            </geometry>
-        </visual>
-        <collision>
-            <geometry>
-                <mesh filename="file://$(find moveit_resources_panda_description)/meshes/collision/link5.stl" />
+                <mesh filename="file://$(find panda_description)/meshes/visual/link5.dae" />
+            </geometry>
+        </visual>
+        <collision>
+            <geometry>
+                <mesh filename="file://$(find panda_description)/meshes/collision/link5.stl" />
             </geometry>
         </collision>
@@ -155,10 +155,10 @@
         <visual>
             <geometry>
-                <mesh filename="file://$(find moveit_resources_panda_description)/meshes/visual/link6.dae" />
-            </geometry>
-        </visual>
-        <collision>
-            <geometry>
-                <mesh filename="file://$(find moveit_resources_panda_description)/meshes/collision/link6.stl" />
+                <mesh filename="file://$(find panda_description)/meshes/visual/link6.dae" />
+            </geometry>
+        </visual>
+        <collision>
+            <geometry>
+                <mesh filename="file://$(find panda_description)/meshes/collision/link6.stl" />
             </geometry>
         </collision>
@@ -181,10 +181,10 @@
         <visual>
             <geometry>
-                <mesh filename="file://$(find moveit_resources_panda_description)/meshes/visual/link7.dae" />
-            </geometry>
-        </visual>
-        <collision>
-            <geometry>
-                <mesh filename="file://$(find moveit_resources_panda_description)/meshes/collision/link7.stl" />
+                <mesh filename="file://$(find panda_description)/meshes/visual/link7.dae" />
+            </geometry>
+        </visual>
+        <collision>
+            <geometry>
+                <mesh filename="file://$(find panda_description)/meshes/collision/link7.stl" />
             </geometry>
         </collision>
@@ -219,10 +219,10 @@
         <visual>
             <geometry>
-                <mesh filename="file://$(find moveit_resources_panda_description)/meshes/visual/hand.dae" />
-            </geometry>
-        </visual>
-        <collision>
-            <geometry>
-                <mesh filename="file://$(find moveit_resources_panda_description)/meshes/collision/hand.stl" />
+                <mesh filename="file://$(find panda_description)/meshes/visual/hand.dae" />
+            </geometry>
+        </visual>
+        <collision>
+            <geometry>
+                <mesh filename="file://$(find panda_description)/meshes/collision/hand.stl" />
             </geometry>
         </collision>
@@ -236,10 +236,10 @@
         <visual>
             <geometry>
-                <mesh filename="file://$(find moveit_resources_panda_description)/meshes/visual/finger.dae" />
-            </geometry>
-        </visual>
-        <collision>
-            <geometry>
-                <mesh filename="file://$(find moveit_resources_panda_description)/meshes/collision/finger.stl" />
+                <mesh filename="file://$(find panda_description)/meshes/visual/finger.dae" />
+            </geometry>
+        </visual>
+        <collision>
+            <geometry>
+                <mesh filename="file://$(find panda_description)/meshes/collision/finger.stl" />
             </geometry>
         </collision>
@@ -254,5 +254,5 @@
             <origin rpy="0 0 3.14159265359" xyz="0 0 0" />
             <geometry>
-                <mesh filename="file://$(find moveit_resources_panda_description)/meshes/visual/finger.dae" />
+                <mesh filename="file://$(find panda_description)/meshes/visual/finger.dae" />
             </geometry>
         </visual>
@@ -260,5 +260,5 @@
             <origin rpy="0 0 3.14159265359" xyz="0 0 0" />
             <geometry>
-                <mesh filename="file://$(find moveit_resources_panda_description)/meshes/collision/finger.stl" />
+                <mesh filename="file://$(find panda_description)/meshes/collision/finger.stl" />
             </geometry>
         </collision>
