Commit message: More Progress on Po, almost getting gripper to work

File: Control/panda/src/panda_description/urdf/backup.urdf.xacro (robot description, xacro)
@@ -1,3 +1,3 @@
-<?xml version="2.0" ?>
+<?xml version="1.0" ?>
 <!-- =================================================================================== -->
 <!-- |    This document was autogenerated by xacro from /opt/ros/kinetic/share/moveit_resources/panda_description/urdf/panda.urdf | -->

File: Control/panda/src/panda_description/urdf/panda_desc.urdf.xacro (robot description, xacro)
@@ -5,4 +5,10 @@
 <!-- =================================================================================== -->
 <robot name="panda" xmlns:xacro="http://www.ros.org/wiki/xacro">
+		<link name="world">
+		</link>
+		<joint name="world_joint" type="fixed">
+			<parent link="world"/>
+			<child link="base_link"/>
+		</joint>
     <link name="base_link">
       <inertial>
