Commit message: The Legend of Po finally works, in gazebo that is, moveit next

File: Control/panda/src/panda_description/urdf/ros2_control.xacro (robot description, xacro)
@@ -56,4 +56,6 @@
             </joint>
             <joint name="panda_finger_joint1">
+								<param name="mimic">panda_finger_joint2</param>
+								<param name="multiplier">1</param>
                 <command_interface name="position"/>
                 <state_interface name="position">

File: Control/panda/src/panda_description_moveit_config/config/panda.ros2_control.xacro (robot description, xacro)
@@ -64,4 +64,11 @@
                 <state_interface name="velocity"/>
             </joint>
+            <joint name="panda_finger_joint2">
+                <command_interface name="position"/>
+                <state_interface name="position">
+                  <param name="initial_value">${initial_positions['panda_finger_joint1']}</param>
+                </state_interface>
+                <state_interface name="velocity"/>
+            </joint>
         </ros2_control>
     </xacro:macro>
