Commit message: more po stuff

File: Control/moveit2_UR5/src/robot_description/urdf/ur5.urdf.xacro (robot description, xacro)
@@ -69,17 +69,17 @@
       <visual>
         <geometry>
-          <mesh filename="package://robot_description/meshes/ur5/visual/base.dae" />
-        </geometry>
-        <material name="LightGrey">
-          <color rgba="0.7 0.7 0.7 1.0"/>
-        </material>
-      </visual>
-      <collision>
-        <geometry>
-          <mesh filename="package://robot_description/meshes/ur5/collision/base.stl" />
+          <mesh filename="$(find robot_description)/meshes/ur5/visual/base.dae" />
+        </geometry>
+        <material name="LightGrey">
+          <color rgba="0.7 0.7 0.7 1.0"/>
+        </material>
+      </visual>
+      <collision>
+        <geometry>
+          <mesh filename="$(find robot_description)/meshes/ur5/collision/base.stl" />
         </geometry>
       </collision>
       <xacro:cylinder_inertial radius="0.1" length="0.15" mass="${base_mass}">
-        <origin xyz="0.0 0.0 0.0" rpy="0 0 0" />
+        <origin xyz="0.0 0.0 10" rpy="0 0 0" />
       </xacro:cylinder_inertial>
     </link>
@@ -100,13 +100,13 @@
       <visual>
         <geometry>
-          <mesh filename="package://robot_description/meshes/ur5/visual/shoulder.dae" />
-        </geometry>
-        <material name="LightGrey">
-          <color rgba="0.7 0.7 0.7 1.0"/>
-        </material>
-      </visual>
-      <collision>
-        <geometry>
-          <mesh filename="package://robot_description/meshes/ur5/collision/shoulder.stl" />
+          <mesh filename="$(find robot_description)/meshes/ur5/visual/shoulder.dae" />
+        </geometry>
+        <material name="LightGrey">
+          <color rgba="0.7 0.7 0.7 1.0"/>
+        </material>
+      </visual>
+      <collision>
+        <geometry>
+          <mesh filename="$(find robot_description)/meshes/ur5/collision/shoulder.stl" />
         </geometry>
       </collision>
@@ -131,13 +131,13 @@
       <visual>
         <geometry>
-          <mesh filename="package://robot_description/meshes/ur5/visual/upperarm.dae" />
-        </geometry>
-        <material name="LightGrey">
-          <color rgba="0.7 0.7 0.7 1.0"/>
-        </material>
-      </visual>
-      <collision>
-        <geometry>
-          <mesh filename="package://robot_description/meshes/ur5/collision/upperarm.stl" />
+          <mesh filename="$(find robot_description)/meshes/ur5/visual/upperarm.dae" />
+        </geometry>
+        <material name="LightGrey">
+          <color rgba="0.7 0.7 0.7 1.0"/>
+        </material>
+      </visual>
+      <collision>
+        <geometry>
+          <mesh filename="$(find robot_description)/meshes/ur5/collision/upperarm.stl" />
         </geometry>
       </collision>
@@ -162,13 +162,13 @@
       <visual>
         <geometry>
-          <mesh filename="package://robot_description/meshes/ur5/visual/forearm.dae" />
-        </geometry>
-        <material name="LightGrey">
-          <color rgba="0.7 0.7 0.7 1.0"/>
-        </material>
-      </visual>
-      <collision>
-        <geometry>
-          <mesh filename="package://robot_description/meshes/ur5/collision/forearm.stl" />
+          <mesh filename="$(find robot_description)/meshes/ur5/visual/forearm.dae" />
+        </geometry>
+        <material name="LightGrey">
+          <color rgba="0.7 0.7 0.7 1.0"/>
+        </material>
+      </visual>
+      <collision>
+        <geometry>
+          <mesh filename="$(find robot_description)/meshes/ur5/collision/forearm.stl" />
         </geometry>
       </collision>
@@ -193,13 +193,13 @@
       <visual>
         <geometry>
-          <mesh filename="package://robot_description/meshes/ur5/visual/wrist1.dae" />
-        </geometry>
-        <material name="LightGrey">
-          <color rgba="0.7 0.7 0.7 1.0"/>
-        </material>
-      </visual>
-      <collision>
-        <geometry>
-          <mesh filename="package://robot_description/meshes/ur5/collision/wrist1.stl" />
+          <mesh filename="$(find robot_description)/meshes/ur5/visual/wrist1.dae" />
+        </geometry>
+        <material name="LightGrey">
+          <color rgba="0.7 0.7 0.7 1.0"/>
+        </material>
+      </visual>
+      <collision>
+        <geometry>
+          <mesh filename="$(find robot_description)/meshes/ur5/collision/wrist1.stl" />
         </geometry>
       </collision>
@@ -224,13 +224,13 @@
       <visual>
         <geometry>
-          <mesh filename="package://robot_description/meshes/ur5/visual/wrist2.dae" />
-        </geometry>
-        <material name="LightGrey">
-          <color rgba="0.7 0.7 0.7 1.0"/>
-        </material>
-      </visual>
-      <collision>
-        <geometry>
-          <mesh filename="package://robot_description/meshes/ur5/collision/wrist2.stl" />
+          <mesh filename="$(find robot_description)/meshes/ur5/visual/wrist2.dae" />
+        </geometry>
+        <material name="LightGrey">
+          <color rgba="0.7 0.7 0.7 1.0"/>
+        </material>
+      </visual>
+      <collision>
+        <geometry>
+          <mesh filename="$(find robot_description)/meshes/ur5/collision/wrist2.stl" />
         </geometry>
       </collision>
@@ -255,13 +255,13 @@
       <visual>
         <geometry>
-          <mesh filename="package://robot_description/meshes/ur5/visual/wrist3.dae" />
-        </geometry>
-        <material name="LightGrey">
-          <color rgba="0.7 0.7 0.7 1.0"/>
-        </material>
-      </visual>
-      <collision>
-        <geometry>
-          <mesh filename="package://robot_description/meshes/ur5/collision/wrist3.stl" />
+          <mesh filename="$(find robot_description)/meshes/ur5/visual/wrist3.dae" />
+        </geometry>
+        <material name="LightGrey">
+          <color rgba="0.7 0.7 0.7 1.0"/>
+        </material>
+      </visual>
+      <collision>
+        <geometry>
+          <mesh filename="$(find robot_description)/meshes/ur5/collision/wrist3.stl" />
         </geometry>
       </collision>

File: Control/panda/src/panda_description/urdf/panda.urdf.xacro (robot description, xacro)
@@ -1,5 +1,5 @@
 <?xml version="1.0" ?>
 <robot name="panda" xmlns:xacro="http://www.ros.org/wiki/xacro">
-  <xacro:include filename="$(find panda_description)/urdf/panda_desc2.urdf.xacro" />
+  <xacro:include filename="$(find panda_description)/urdf/panda_desc.urdf.xacro" />
   <xacro:include filename="$(find panda_description)/urdf/panda.gazebo" />
   <xacro:include filename="$(find panda_description)/urdf/ros2_control.xacro" />
