Commit message: more po stuff

File: Control/panda/src/panda_description/urdf/panda_desc.urdf.xacro (robot description, xacro)
@@ -5,290 +5,340 @@
 <!-- =================================================================================== -->
 <robot name="panda" xmlns:xacro="http://www.ros.org/wiki/xacro">
-		<link name="world">
-		</link>
     <link name="base_link">
-        <visual>
-            <geometry>
-                <mesh filename="file://$(find panda_description)/meshes/visual/link0.dae" />
-            </geometry>
-        </visual>
-        <collision>
-            <geometry>
-                <mesh filename="file://$(find panda_description)/meshes/collision/link0.stl" />
-            </geometry>
-        </collision>
-        <inertial>
-          <origin xyz="-0.041018 -0.00014 0.049974" rpy="0 0 0" />
-          <mass value="0.629769"/>
-          <inertia ixx="0.00315" iyy="0.00388" izz="0.004285" ixy="8.2904E-7" ixz="0.00015" iyz="8.2299E-6"/>
-        </inertial>
-    </link>
+      <inertial>
+        <mass value="2.92"/>
+        <origin rpy="0 0 0" xyz="-0.025566 -2.88e-05 0.057332"/>
+        <inertia ixx="0.00782229414331" ixy="-1.56191622996e-05" ixz="-0.00126005738123" iyy="0.0109027971813" iyz="1.08233858202e-05" izz="0.0102355503949"/>
+      </inertial>
+      <visual>
+        <origin rpy="0 0 0" xyz="0 0 0"/>
+        <geometry>
+          <mesh filename="file://$(find panda_description)/meshes/visual/link0.dae"/>
+        </geometry>
+        <material name="">
+          <color rgba="1 1 1 1"/>
+        </material>
+      </visual>
+      <collision>
+        <origin rpy="0 0 0" xyz="0 0 0"/>
+        <geometry>
+          <mesh filename="file://$(find panda_description)/meshes/collision/link0.stl"/>
+        </geometry>
+      </collision>
+    </link>
+    <!-- panda_link1 -->
     <link name="panda_link1">
-        <visual>
-            <geometry>
-                <mesh filename="file://$(find panda_description)/meshes/visual/link1.dae" />
-            </geometry>
-        </visual>
-        <collision>
-            <geometry>
-                <mesh filename="file://$(find panda_description)/meshes/collision/link1.stl" />
-            </geometry>
-        </collision>
-        <inertial>
-          <origin xyz="0.003875 0.002081 -0.04762" rpy="0 0 0" />
-          <mass value="4.970684"/>
-          <inertia ixx="0.70337" iyy="0.70661" izz="0.009117" ixy="-0.000139" ixz="0.006772" iyz="0.019169"/>
-        </inertial>
-    </link>
-		<joint name="world_joint" type="fixed">
-			<parent link="world"/>
-			<child link="base_link"/>
-		</joint>
+      <inertial>
+        <mass value="2.74"/>
+        <origin rpy="0 0 0" xyz="0 -0.0324958 -0.0675818"/>
+        <inertia ixx="0.0180416958283" ixy="0.0" ixz="0.0" iyy="0.0159136071891" iyz="0.0046758424612" izz="0.00620690827127"/>
+      </inertial>
+      <visual>
+        <origin rpy="0 0 0" xyz="0 0 0"/>
+        <geometry>
+          <mesh filename="file://$(find panda_description)/meshes/visual/link1.dae"/>
+        </geometry>
+        <material name="">
+          <color rgba="1 1 1 1"/>
+        </material>
+      </visual>
+      <collision>
+        <origin rpy="0 0 0" xyz="0 0 0"/>
+        <geometry>
+          <mesh filename="file://$(find panda_description)/meshes/collision/link1.stl"/>
+        </geometry>
+      </collision>
+    </link>
+    <!-- panda_joint1 -->
     <joint name="panda_joint1" type="revolute">
-        <safety_controller k_position="100.0" k_velocity="40.0" soft_lower_limit="-2.8973" soft_upper_limit="2.8973" />
-        <origin rpy="0 0 0" xyz="0 0 0.333" />
-        <parent link="base_link" />
-        <child link="panda_link1" />
-        <axis xyz="0 0 1" />
-        <limit effort="87" lower="-2.9671" upper="2.9671" velocity="2.3925" />
-        <dynamics D="1" K="7000" damping="0.003" friction="0.0" mu_coulomb="0" mu_viscous="16" />
-    </joint>
+      <origin rpy="0 0 0" xyz="0 0 0.333"/>
+      <parent link="base_link"/>
+      <child link="panda_link1"/>
+      <axis xyz="0 0 1"/>
+      <limit effort="87" lower="-2.8973" upper="2.8973" velocity="2.1750"/>
+    </joint>
+    <!-- panda_link2 -->
     <link name="panda_link2">
-        <visual>
-            <geometry>
-                <mesh filename="file://$(find panda_description)/meshes/visual/link2.dae" />
-            </geometry>
-        </visual>
-        <collision>
-            <geometry>
-                <mesh filename="file://$(find panda_description)/meshes/collision/link2.stl" />
-            </geometry>
-        </collision>
-        <inertial>
-          <origin xyz="-0.003141 -0.02872  0.003495" rpy="0 0 0" />
-          <mass value="0.646926"/>
-          <inertia ixx="0.007962" iyy="2.811E-2" izz="2.5995E-2" ixy="-3.925E-3" ixz="1.0254E-2" iyz="7.04E-4"/>
-        </inertial>
-    </link>
+      <inertial>
+        <mass value="2.74"/>
+        <origin rpy="0 0 0" xyz="0 -0.06861 0.0322285"/>
+        <inertia ixx="0.0182856182281" ixy="0.0" ixz="0.0" iyy="0.00621358421175" iyz="-0.00472844221905" izz="0.0161514346309"/>
+      </inertial>
+      <visual>
+        <origin rpy="0 0 0" xyz="0 0 0"/>
+        <geometry>
+          <mesh filename="file://$(find panda_description)/meshes/visual/link2.dae"/>
+        </geometry>
+        <material name="">
+          <color rgba="1 1 1 1"/>
+        </material>
+      </visual>
+      <collision>
+        <origin rpy="0 0 0" xyz="0 0 0"/>
+        <geometry>
+          <mesh filename="file://$(find panda_description)/meshes/collision/link2.stl"/>
+        </geometry>
+      </collision>
+    </link>
+    <!-- panda_joint2 -->
     <joint name="panda_joint2" type="revolute">
-        <safety_controller k_position="100.0" k_velocity="40.0" soft_lower_limit="-1.7628" soft_upper_limit="1.7628" />
-        <origin rpy="-1.57079632679 0 0" xyz="0 0 0" />
-        <parent link="panda_link1" />
-        <child link="panda_link2" />
-        <axis xyz="0 0 1" />
-        <limit effort="87" lower="-1.8326" upper="1.8326" velocity="2.3925" />
-        <dynamics D="1" K="7000" damping="0.003" friction="0.0" mu_coulomb="0" mu_viscous="16" />
-    </joint>
+      <origin rpy="-1.57079632679 0 0" xyz="0 0 0"/>
+      <parent link="panda_link1"/>
+      <child link="panda_link2"/>
+      <axis xyz="0 0 1"/>
+      <limit effort="87" lower="-1.7628" upper="1.7628" velocity="2.1750"/>
+    </joint>
+    <!-- panda_link3 -->
     <link name="panda_link3">
-        <visual>
-            <geometry>
-                <mesh filename="file://$(find panda_description)/meshes/visual/link3.dae" />
-            </geometry>
-        </visual>
-        <collision>
-            <geometry>
-                <mesh filename="file://$(find panda_description)/meshes/collision/link3.stl" />
-            </geometry>
-        </collision>
-        <inertial>
-          <origin xyz="2.7518E-2 3.9252E-2 -6.6502E-2" rpy="0 0 0" />
-          <mass value="3.228604"/>
-          <inertia ixx="3.7242E-2" iyy="3.6155E-2" izz="1.083E-2" ixy="-4.761E-3" ixz="-1.1396E-2" iyz="-1.2805E-2"/>
-        </inertial>
-    </link>
+      <inertial>
+        <mass value="2.38"/>
+        <origin rpy="0 0 0" xyz="0.0469893 0.0316374 -0.031704"/>
+        <inertia ixx="0.00771376630908" ixy="-0.00248490625138" ixz="-0.00332147581033" iyy="0.00989108008727" iyz="-0.00217796151484" izz="0.00811723558464"/>
+      </inertial>
+      <visual>
+        <origin rpy="0 0 0" xyz="0 0 0"/>
+        <geometry>
+          <mesh filename="file://$(find panda_description)/meshes/visual/link3.dae"/>
+        </geometry>
+        <material name="">
+          <color rgba="1 1 1 1"/>
+        </material>
+      </visual>
+      <collision>
+        <origin rpy="0 0 0" xyz="0 0 0"/>
+        <geometry>
+          <mesh filename="file://$(find panda_description)/meshes/collision/link3.stl"/>
+        </geometry>
+      </collision>
+    </link>
+    <!-- panda_joint3 -->
     <joint name="panda_joint3" type="revolute">
-        <safety_controller k_position="100.0" k_velocity="40.0" soft_lower_limit="-2.8973" soft_upper_limit="2.8973" />
-        <origin rpy="1.57079632679 0 0" xyz="0 -0.316 0" />
-        <parent link="panda_link2" />
-        <child link="panda_link3" />
-        <axis xyz="0 0 1" />
-        <limit effort="87" lower="-2.9671" upper="2.9671" velocity="2.3925" />
-        <dynamics D="1" K="7000" damping="0.003" friction="0.0" mu_coulomb="0" mu_viscous="16" />
-    </joint>
+      <origin rpy="1.57079632679 0 0" xyz="0 -0.316 0"/>
+      <parent link="panda_link2"/>
+      <child link="panda_link3"/>
+      <axis xyz="0 0 1"/>
+      <limit effort="87" lower="-2.8973" upper="2.8973" velocity="2.1750"/>
+    </joint>
+    <!-- panda_link4-->
     <link name="panda_link4">
-        <visual>
-            <geometry>
-                <mesh filename="file://$(find panda_description)/meshes/visual/link4.dae" />
-            </geometry>
-        </visual>
-        <collision>
-            <geometry>
-                <mesh filename="file://$(find panda_description)/meshes/collision/link4.stl" />
-            </geometry>
-        </collision>
-        <inertial>
-          <origin xyz="-5.317E-2 1.04419E-1 2.7454E-2" rpy="0 0 0" />
-          <mass value="3.587895"/>
-          <inertia ixx="2.5853E-2" iyy="1.9552E-2" izz="2.8323E-2" ixy="7.796E-3" ixz="-1.332E-3" iyz="8.641E-3"/>
-        </inertial>
-    </link>
+      <inertial>
+        <mass value="2.38"/>
+        <origin rpy="0 0 0" xyz="-0.0360446 0.0336853 0.031882"/>
+        <inertia ixx="0.00799663881132" ixy="0.00347095570217" ixz="-0.00241222942995" iyy="0.00825390705278" iyz="0.00235774044121" izz="0.0102515004345"/>
+      </inertial>
+      <visual>
+        <origin rpy="0 0 0" xyz="0 0 0"/>
+        <geometry>
+          <mesh filename="file://$(find panda_description)/meshes/visual/link4.dae"/>
+        </geometry>
+        <material name="">
+          <color rgba="1 1 1 1"/>
+        </material>
+      </visual>
+      <collision>
+        <origin rpy="0 0 0" xyz="0 0 0"/>
+        <geometry>
+          <mesh filename="file://$(find panda_description)/meshes/collision/link4.stl"/>
+        </geometry>
+      </collision>
+    </link>
+    <!-- panda_joint4 -->
     <joint name="panda_joint4" type="revolute">
-        <safety_controller k_position="100.0" k_velocity="40.0" soft_lower_limit="-3.0718" soft_upper_limit="0.0175" />
-        <origin rpy="1.57079632679 0 0" xyz="0.0825 0 0" />
-        <parent link="panda_link3" />
-        <child link="panda_link4" />
-        <axis xyz="0 0 1" />
-        <limit effort="87" lower="-3.1416" upper="0.0873" velocity="2.3925" />
-        <dynamics D="1" K="7000" damping="0.003" friction="0.0" mu_coulomb="0" mu_viscous="16" />
-    </joint>
+      <origin rpy="1.57079632679 0 0" xyz="0.0825 0 0"/>
+      <parent link="panda_link3"/>
+      <child link="panda_link4"/>
+      <axis xyz="0 0 1"/>
+      <limit effort="87" lower="-3.0718" upper="0.0698" velocity="2.1750"/>
+      <!-- upper should be -0.0698, but that brakes simulation when initial position for this joint is 0.0 -->
+    </joint>
+    <!-- panda_link5 -->
     <link name="panda_link5">
-        <visual>
-            <geometry>
-                <mesh filename="file://$(find panda_description)/meshes/visual/link5.dae" />
-            </geometry>
-        </visual>
-        <collision>
-            <geometry>
-                <mesh filename="file://$(find panda_description)/meshes/collision/link5.stl" />
-            </geometry>
-        </collision>
-        <inertial>
-          <origin xyz="-1.1953E-2 4.1065E-2 -3.8437E-2" rpy="0 0 0" />
-          <mass value="1.225946"/>
-          <inertia ixx="3.5549E-2" iyy="2.9474E-2" izz="8.627E-3" ixy="-2.117E-3" ixz="-4.037E-3" iyz="2.29E-4"/>
-        </inertial>
-    </link>
+      <inertial>
+        <mass value="2.74"/>
+        <origin rpy="0 0 0" xyz="0 0.0610427 -0.104176"/>
+        <inertia ixx="0.030371374513" ixy="6.50283587108e-07" ixz="-1.05129179916e-05" iyy="0.0288752887402" iyz="-0.00775653445787" izz="0.00444134056164"/>
+      </inertial>
+      <visual>
+        <origin rpy="0 0 0" xyz="0 0 0"/>
+        <geometry>
+          <mesh filename="file://$(find panda_description)/meshes/visual/link5.dae"/>
+        </geometry>
+        <material name="">
+          <color rgba="1 1 1 1"/>
+        </material>
+      </visual>
+      <collision>
+        <origin rpy="0 0 0" xyz="0 0 0"/>
+        <geometry>
+          <mesh filename="file://$(find panda_description)/meshes/collision/link5.stl"/>
+        </geometry>
+      </collision>
+    </link>
+    <!-- panda_joint5 -->
     <joint name="panda_joint5" type="revolute">
-        <safety_controller k_position="100.0" k_velocity="40.0" soft_lower_limit="-2.8973" soft_upper_limit="2.8973" />
-        <origin rpy="-1.57079632679 0 0" xyz="-0.0825 0.384 0" />
-        <parent link="panda_link4" />
-        <child link="panda_link5" />
-        <axis xyz="0 0 1" />
-        <limit effort="12" lower="-2.9671" upper="2.9671" velocity="2.8710" />
-        <dynamics D="1" K="7000" damping="0.003" friction="0.0" mu_coulomb="0" mu_viscous="16" />
-    </joint>
+      <origin rpy="-1.57079632679 0 0" xyz="-0.0825 0.384 0"/>
+      <parent link="panda_link4"/>
+      <child link="panda_link5"/>
+      <axis xyz="0 0 1"/>
+      <limit effort="12" lower="-2.8973" upper="2.8973" velocity="2.6100"/>
+    </joint>
+    <!-- panda_link6 -->
     <link name="panda_link6">
-        <visual>
-            <geometry>
-                <mesh filename="file://$(find panda_description)/meshes/visual/link6.dae" />
-            </geometry>
-        </visual>
-        <collision>
-            <geometry>
-                <mesh filename="file://$(find panda_description)/meshes/collision/link6.stl" />
-            </geometry>
-        </collision>
-        <inertial>
-          <origin xyz="6.0149E-2 -1.4117E-2 -1.0517E-2" rpy="0 0 0" />
-          <mass value="1.666555"/>
-          <inertia ixx="1.964E-3" iyy="4.354E-3" izz="5.433E-3" ixy="1.09E-4" ixz="-1.158E-3" iyz="3.41E-4"/>
-        </inertial>
-    </link>
+      <inertial>
+        <mass value="1.55"/>
+        <origin rpy="0 0 0" xyz="0.0510509 0.009108 0.0106343"/>
+        <inertia ixx="0.00303336450376" ixy="-0.000437276865508" ixz="0.000629257294877" iyy="0.00404479911567" iyz="0.000130472021025" izz="0.00558234286039"/>
+      </inertial>
+      <visual>
+        <origin rpy="0 0 0" xyz="0 0 0"/>
+        <geometry>
+          <mesh filename="file://$(find panda_description)/meshes/visual/link6.dae"/>
+        </geometry>
+        <material name="">
+          <color rgba="1 1 1 1"/>
+        </material>
+      </visual>
+      <collision>
+        <origin rpy="0 0 0" xyz="0 0 0"/>
+        <geometry>
+          <mesh filename="file://$(find panda_description)/meshes/collision/link6.stl"/>
+        </geometry>
+      </collision>
+    </link>
+    <!-- panda_joint6 -->
     <joint name="panda_joint6" type="revolute">
-        <safety_controller k_position="100.0" k_velocity="40.0" soft_lower_limit="-0.0175" soft_upper_limit="3.7525" />
-        <origin rpy="1.57079632679 0 0" xyz="0 0 0" />
-        <parent link="panda_link5" />
-        <child link="panda_link6" />
-        <axis xyz="0 0 1" />
-        <limit effort="12" lower="-0.0873" upper="3.8223" velocity="2.8710" />
-        <dynamics D="1" K="7000" damping="0.003" friction="0.0" mu_coulomb="0" mu_viscous="16" />
-    </joint>
+      <origin rpy="1.57079632679 -1.57079632679 0" xyz="0 0 0"/> <!-- rpy="1.57079632679 0 0" -->
+      <parent link="panda_link5"/>
+      <child link="panda_link6"/>
+      <axis xyz="0 0 1"/>
+      <limit effort="12" lower="-0.0175" upper="3.7525" velocity="2.6100"/>
+    </joint>
+    <!-- panda_link7 -->
     <link name="panda_link7">
-        <visual>
-            <geometry>
-                <mesh filename="file://$(find panda_description)/meshes/visual/link7.dae" />
-            </geometry>
-        </visual>
-        <collision>
-            <geometry>
-                <mesh filename="file://$(find panda_description)/meshes/collision/link7.stl" />
-            </geometry>
-        </collision>
-        <inertial>
-          <origin xyz="1.0517E-2 -4.252E-3 6.1597E-2" rpy="0 0 0" />
-          <mass value="7.35522E-1"/>
-          <inertia ixx="1.2516E-2" iyy="1.0027E-2" izz="4.815E-3" ixy="-4.28E-4" ixz="-1.19E-3" iyz="-7.41E-4"/>
-        </inertial>
-    </link>
+      <inertial>
+        <mass value="0.54"/>
+        <origin rpy="0 0 0" xyz="0.0109695 0.0107965 0.0650411"/>
+        <inertia ixx="0.000888868887021" ixy="-0.00012239074652" ixz="3.98699829666e-05" iyy="0.000888001373233" iyz="-9.33825115206e-05" izz="0.0007176834609"/>
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